Commit message: Created new launch file, 3_agents_moving_awayLine.launch, which spawns in 3 agents. After launching, publish true to the /control_on topic to get the agents to move. Also fixed an issue where turtlebots would slowly turn in place (multiplied wheel masses by 10x and inertias by 100x as per internet forum). Also fixed an issue in the consensus where data could be changed mid-consensus (added mutex lock)

File: dse_turtlebot_descriptions/urdf/turtlebot3_burger.urdf.xacro (robot description, xacro)
@@ -57,8 +57,8 @@
     <inertial>
       <origin xyz="0 0 0" />
-      <mass value="2.8498940e-02" />
-      <inertia ixx="1.1175580e-05" ixy="-4.2369783e-11" ixz="-5.9381719e-09"
-               iyy="1.1192413e-05" iyz="-1.4400107e-11"
-               izz="2.0712558e-05" />
+      <mass value="2.8498940e-01" />
+      <inertia ixx="1.1175580e-03" ixy="-4.2369783e-9" ixz="-5.9381719e-07"
+               iyy="1.1192413e-03" iyz="-1.4400107e-9"
+               izz="2.0712558e-03" />
       </inertial>
   </link>
@@ -85,8 +85,8 @@
     <inertial>
       <origin xyz="0 0 0" />
-      <mass value="2.8498940e-02" />
-      <inertia ixx="1.1175580e-05" ixy="-4.2369783e-11" ixz="-5.9381719e-09"
-               iyy="1.1192413e-05" iyz="-1.4400107e-11"
-               izz="2.0712558e-05" />
+      <mass value="2.8498940e-01" />
+      <inertia ixx="1.1175580e-03" ixy="-4.2369783e-9" ixz="-5.9381719e-07"
+               iyy="1.1192413e-03" iyz="-1.4400107e-9"
+               izz="2.0712558e-03" />
       </inertial>
   </link>

Commit message: Changed pose_markers message to used array of PoseStamped and started working on a circular simulation. NOTE - Agents have their camera facing left right now.

File: dse_turtlebot_descriptions/urdf/turtlebot3_burger.urdf.xacro (robot description, xacro)
@@ -145,5 +145,5 @@
   </link>
   <joint name="camera_joint" type="fixed">
-    <origin xyz="0.064 -0.065 0.094" rpy="0 0 0"/>
+    <origin xyz="0.064 -0.065 0.094" rpy="0 0 -1.57"/>
     <parent link="base_link"/>
     <child link="camera_link"/>

Commit message: Intrinsically and Extrinsically calibrated the aruco estimations. Check the JIRA meeting notes for more details on that.

File: dse_turtlebot_descriptions/urdf/turtlebot3_burger.urdf.xacro (robot description, xacro)
@@ -145,5 +145,7 @@
   </link>
   <joint name="camera_joint" type="fixed">
-    <origin xyz="0.064 -0.065 0.094" rpy="0 0 -1.57"/>
+    <origin xyz="0.064 -0.065 0.094" rpy="0 0 0"/>
+    <!-- Noramal: <origin xyz="0.064 -0.065 0.094" rpy="0 0 0"/>-->
+    <!-- Turned right: <origin xyz="0.064 -0.065 0.094" rpy="0 0 -1.57"/>-->
     <parent link="base_link"/>
     <child link="camera_link"/>
